Commit message: sync: new_urdf 资源基线 + damping_0_reward_v1+symmerty（joint_symmetry 镜像对称奖励治偏航）
- 资源基线: lumber_* -> lumbar_* 重命名 + 新增 Camera/head/neck/radar meshes + mjcf X1_12DOF 系列 + x1.urdf 更新

- x1_dh_stand_config.py: heading_command True->False（yaw 稳定改由 joint_symmetry 承担）；foot_slip -0.1->-1.0；新增 joint_symmetry = 0.8

- x1_dh_stand_env.py: 接触判定阈值 5->40N（3 处）；foot_slip sqrt->线性；feet_contact_number 失配惩罚 -0.3->-1.0；新增 _reward_joint_symmetry（hip_roll/hip_yaw/ankle_roll L+R 镜像和约束，|yaw_cmd|>0.15 turning 门控）

- play.py: heading_command 与训练一致设为 False

v7 sim 证据: heading=False + symmetry -> yaw rate 0.61 deg/s（无约束 -2.75）；真机 20260818 all-rv1 yaw drift +13.9 deg/s 待治

File: resources/robots/x1/urdf/x1.urdf (robot description, URDF)
Before this commit: robot x1, 58 links, 57 joints
Links:
- removed link arm_l_wrist_a_ball
- removed link arm_l_wrist_a_loop
- removed link arm_l_wrist_b_ball
- removed link arm_l_wrist_b_loop
- removed link arm_r_wrist_a_ball
- removed link arm_r_wrist_a_loop
- removed link arm_r_wrist_b_ball
- removed link arm_r_wrist_b_loop
- removed link left_ankle_pitch
- removed link left_ankle_roll
- removed link left_elbow_pitch
- removed link left_elbow_yaw
- removed link left_hip_pitch
- removed link left_hip_roll
- removed link left_hip_yaw
- removed link left_knee_pitch
- removed link left_shoulder_pitch
- removed link left_shoulder_roll
- removed link left_shoulder_yaw
- removed link left_wrist_pitch
- removed link leg_l_toe_a_ball
- removed link leg_l_toe_a_loop
- removed link leg_l_toe_b_ball
- removed link leg_l_toe_b_loop
- removed link leg_r_toe_a_ball
- removed link leg_r_toe_a_loop
- removed link leg_r_toe_b_ball
- removed link leg_r_toe_b_loop
- removed link lumber_pitch
- removed link lumber_roll
- removed link lumber_yaw
- removed link right_ankle_pitch
- removed link right_ankle_roll
- removed link right_elbow_pitch
- removed link right_elbow_yaw
- removed link right_hip_pitch
- removed link right_hip_roll
- removed link right_hip_yaw
- removed link right_knee_pitch
- removed link right_shoulder_pitch
- removed link right_shoulder_roll
- removed link right_shoulder_yaw
- removed link right_wrist_pitch
- removed link waist_motor_a_ball
- removed link waist_motor_a_loop
- removed link waist_motor_b_ball
- removed link waist_motor_b_loop
- added link arm_l_wrist_a_ball_link, mass 0.23598732; visual mesh filename=../meshes/arm_r_wrist_a_ball.STL
- added link arm_l_wrist_a_loop_link, mass 0.00548041; visual mesh filename=../meshes/arm_r_wrist_a_loop.STL
- added link arm_l_wrist_b_ball_link, mass 0.03617567; visual mesh filename=../meshes/arm_r_wrist_b_ball.STL
- added link arm_l_wrist_b_loop_link, mass 0.00117982; visual mesh filename=../meshes/arm_r_wrist_b_loop.STL
- added link arm_r_wrist_a_ball_link, mass 0.23598732; visual mesh filename=../meshes/arm_r_wrist_a_ball.STL
- added link arm_r_wrist_a_loop_link, mass 0.00548041; visual mesh filename=../meshes/arm_r_wrist_a_loop.STL
- added link arm_r_wrist_b_ball_link, mass 0.03617567; visual mesh filename=../meshes/arm_r_wrist_b_ball.STL
- added link arm_r_wrist_b_loop_link, mass 0.00117982; visual mesh filename=../meshes/arm_r_wrist_b_loop.STL
- added link left_ankle_pitch_link, mass 0.06217211; visual mesh filename=../meshes/left_ankle_pitch.STL
- added link left_ankle_roll_link, mass 0.58971207; collision mesh filename=../meshes/left_ankle_roll.STL; visual mesh filename=../meshes/left_ankle_roll.STL
- added link left_elbow_pitch_link, mass 0.69780135; visual mesh filename=../meshes/left_elbow_pitch.STL
- added link left_elbow_yaw_link, mass 0.28787886; visual mesh filename=../meshes/left_elbow_yaw.STL
- added link left_hip_pitch_link, mass 1.6733645; visual mesh filename=../meshes/left_hip_pitch.STL
- added link left_hip_roll_link, mass 0.28562185; visual mesh filename=../meshes/left_hip_roll.STL
- added link left_hip_yaw_link, mass 2.7369623; visual mesh filename=../meshes/left_hip_yaw.STL
- added link left_knee_pitch_link, mass 1.68649; visual mesh filename=../meshes/left_knee_pitch.STL
- added link left_shoulder_pitch_link, mass 1.0067875; visual mesh filename=../meshes/left_shoulder_pitch.STL
- added link left_shoulder_roll_link, mass 0.69169508; visual mesh filename=../meshes/left_shoulder_roll.STL
- added link left_shoulder_yaw_link, mass 0.72559372; visual mesh filename=../meshes/left_shoulder_yaw.STL
- added link left_wrist_pitch_link, mass 0.00900738; visual mesh filename=../meshes/left_wrist_pitch.STL
- added link left_wrist_roll_link, mass 0.370899
- added link leg_l_toe_a_ball_link, mass 0.05674707; visual mesh filename=../meshes/leg_l_toe_a_ball.STL
- added link leg_l_toe_a_loop_link, mass 0.0062017; visual mesh filename=../meshes/leg_l_toe_a_loop.STL
- added link leg_l_toe_b_ball_link, mass 0.0423305; visual mesh filename=../meshes/leg_l_toe_b_ball.STL
- added link leg_l_toe_b_loop_link, mass 0.0062017; visual mesh filename=../meshes/leg_l_toe_b_loop.STL
- added link leg_r_toe_a_ball_link, mass 0.05674707; visual mesh filename=../meshes/leg_r_toe_a_ball.STL
- added link leg_r_toe_a_loop_link, mass 0.0062017; visual mesh filename=../meshes/leg_r_toe_a_loop.STL
- added link leg_r_toe_b_ball_link, mass 0.0423305; visual mesh filename=../meshes/leg_r_toe_b_ball.STL
- added link leg_r_toe_b_loop_link, mass 0.0062017; visual mesh filename=../meshes/leg_r_toe_b_loop.STL
- added link lumbar_pitch_link, mass 8.8571074; visual mesh filename=../meshes/lumbar_pitch_x1.STL
- added link lumbar_roll_link, mass 0.03412073; visual mesh filename=../meshes/lumbar_roll.STL
- added link lumbar_yaw_link, mass 0.36251906; visual mesh filename=../meshes/lumbar_yaw.STL
- added link right_ankle_pitch_link, mass 0.06217211; visual mesh filename=../meshes/right_ankle_pitch.STL
- added link right_ankle_roll_link, mass 0.58971207; collision mesh filename=../meshes/right_ankle_roll.STL; visual mesh filename=../meshes/right_ankle_roll.STL
- added link right_elbow_pitch_link, mass 0.69780135; visual mesh filename=../meshes/right_elbow_pitch.STL
- added link right_elbow_yaw_link, mass 0.28787886; visual mesh filename=../meshes/right_elbow_yaw.STL
- added link right_hip_pitch_link, mass 1.6733645; visual mesh filename=../meshes/right_hip_pitch.STL
- added link right_hip_roll_link, mass 0.28562185; visual mesh filename=../meshes/right_hip_roll.STL
- added link right_hip_yaw_link, mass 2.7369623; visual mesh filename=../meshes/right_hip_yaw.STL
- added link right_knee_pitch_link, mass 1.68649; visual mesh filename=../meshes/right_knee_pitch.STL
- added link right_shoulder_pitch_link, mass 1.0067875; visual mesh filename=../meshes/right_shoulder_pitch.STL
- added link right_shoulder_roll_link, mass 0.69169508; visual mesh filename=../meshes/right_shoulder_roll.STL
- added link right_shoulder_yaw_link, mass 0.72559372; visual mesh filename=../meshes/right_shoulder_yaw.STL
- added link right_wrist_pitch_link, mass 0.00900738; visual mesh filename=../meshes/right_wrist_pitch.STL
- added link right_wrist_roll_link, mass 0.370899
- added link waist_motor_a_ball_link, mass 0.03613902; visual mesh filename=../meshes/waist_motor_a_ball.STL
- added link waist_motor_a_loop_link, mass 0.01765296; visual mesh filename=../meshes/waist_motor_a_loop.STL
- added link waist_motor_b_ball_link, mass 0.03613902; visual mesh filename=../meshes/waist_motor_b_ball.STL
- added link waist_motor_b_loop_link, mass 0.01765296; visual mesh filename=../meshes/waist_motor_b_loop.STL
- link arm_r_wrist_motor_b_link: mass 0.00117982 -> 0.23598732
Joints:
- removed joint lumber_pitch_joint
- removed joint lumber_roll_joint
- removed joint lumber_yaw_joint
- added joint left_wrist_roll_joint: type fixed, parent left_wrist_pitch_link, child left_wrist_roll_link, origin xyz=0 0 0 rpy=-1.4 0.970796 -1.5708
- added joint lumbar_pitch_joint: type fixed, parent lumbar_roll_link, child lumbar_pitch_link, origin xyz=0 0 0 rpy=0 1.5707963267949 0, axis 0 0 -1, limit lower=-3.14 upper=3.14 effort=0 velocity=0
- added joint lumbar_roll_joint: type fixed, parent lumbar_yaw_link, child lumbar_roll_link, origin xyz=0 0 0.0405 rpy=1.57079632679491 0 -1.5707963267949, axis 0 0 1, limit lower=-3.14 upper=3.14 effort=0 velocity=0
- added joint lumbar_yaw_joint: type fixed, parent base_link, child lumbar_yaw_link, origin xyz=0.00244999999994827 0 0.115534033809005 rpy=0 0 -4.54911392613975E-05, axis 0 0 1, limit lower=-3.14 upper=3.14 effort=0 velocity=0
- added joint right_wrist_roll_joint: type fixed, parent right_wrist_pitch_link, child right_wrist_roll_link, origin xyz=0 0 0 rpy=1.74159 0.970796 -1.5708
- joint arm_l_wrist_a_ball_joint: child arm_l_wrist_a_ball -> arm_l_wrist_a_ball_link; parent left_elbow_yaw -> left_elbow_yaw_link
- joint arm_l_wrist_a_loop_joint: child arm_l_wrist_a_loop -> arm_l_wrist_a_loop_link
- joint arm_l_wrist_b_ball_joint: child arm_l_wrist_b_ball -> arm_l_wrist_b_ball_link; parent left_elbow_yaw -> left_elbow_yaw_link
- joint arm_l_wrist_b_loop_joint: child arm_l_wrist_b_loop -> arm_l_wrist_b_loop_link
- joint arm_l_wrist_motor_a_link_joint: parent arm_l_wrist_a_ball -> arm_l_wrist_a_ball_link
- joint arm_l_wrist_motor_b_link_joint: parent arm_l_wrist_b_ball -> arm_l_wrist_b_ball_link
- joint arm_r_wrist_a_ball_joint: child arm_r_wrist_a_ball -> arm_r_wrist_a_ball_link; parent right_elbow_yaw -> right_elbow_yaw_link
- joint arm_r_wrist_a_loop_joint: child arm_r_wrist_a_loop -> arm_r_wrist_a_loop_link
- joint arm_r_wrist_b_ball_joint: child arm_r_wrist_b_ball -> arm_r_wrist_b_ball_link; parent right_elbow_yaw -> right_elbow_yaw_link
- joint arm_r_wrist_b_loop_joint: child arm_r_wrist_b_loop -> arm_r_wrist_b_loop_link
- joint arm_r_wrist_motor_a_link_joint: parent arm_r_wrist_a_ball -> arm_r_wrist_a_ball_link
- joint arm_r_wrist_motor_b_link_joint: parent arm_r_wrist_b_ball -> arm_r_wrist_b_ball_link
- joint left_ankle_pitch_joint: child left_ankle_pitch -> left_ankle_pitch_link; limit lower=-3.14 upper=3.14 effort=80 velocity=10 -> lower=-0.41 upper=0.35 effort=80.0 velocity=13.61; parent left_knee_pitch -> left_knee_pitch_link
- joint left_ankle_roll_joint: child left_ankle_roll -> left_ankle_roll_link; limit lower=-3.14 upper=3.14 effort=80 velocity=10 -> lower=-0.64 upper=0.64 effort=80.0 velocity=13.61; parent left_ankle_pitch -> left_ankle_pitch_link
- joint left_elbow_pitch_joint: child left_elbow_pitch -> left_elbow_pitch_link; parent left_shoulder_yaw -> left_shoulder_yaw_link
- joint left_elbow_yaw_joint: child left_elbow_yaw -> left_elbow_yaw_link; parent left_elbow_pitch -> left_elbow_pitch_link
- joint left_hip_pitch_joint: child left_hip_pitch -> left_hip_pitch_link; limit lower=-3.14 upper=3.14 effort=150 velocity=8 -> lower=-1 upper=2 effort=180 velocity=8.90
- joint left_hip_roll_joint: child left_hip_roll -> left_hip_roll_link; limit lower=-3.14 upper=3.14 effort=150 velocity=8 -> lower=-1.5 upper=0.2 effort=150.0 velocity=27.23; parent left_hip_pitch -> left_hip_pitch_link
- joint left_hip_yaw_joint: child left_hip_yaw -> left_hip_yaw_link; limit lower=-3.14 upper=3.14 effort=50 velocity=24 -> lower=-1.5 upper=1.5 effort=150.0 velocity=27.23; parent left_hip_roll -> left_hip_roll_link
- joint left_knee_pitch_joint: child left_knee_pitch -> left_knee_pitch_link; limit lower=-3.14 upper=3.14 effort=150 velocity=8 -> lower=0 upper=2 effort=180.0 velocity=8.9; parent left_hip_yaw -> left_hip_yaw_link
- joint left_shoulder_pitch_joint: child left_shoulder_pitch -> left_shoulder_pitch_link; parent lumber_pitch -> lumbar_pitch_link
- joint left_shoulder_roll_joint: child left_shoulder_roll -> left_shoulder_roll_link; parent left_shoulder_pitch -> left_shoulder_pitch_link
- joint left_shoulder_yaw_joint: child left_shoulder_yaw -> left_shoulder_yaw_link; parent left_shoulder_roll -> left_shoulder_roll_link
- joint left_wrist_pitch_joint: child left_wrist_pitch -> left_wrist_pitch_link; origin xyz=0.006 9.9998E-05 -0.1394 rpy=1.5708 0 0 -> xyz=0.006 0.0001 -0.1394 rpy=1.5708 0.229204 -1.5708; parent left_elbow_yaw -> left_elbow_yaw_link
- joint leg_l_toe_a_ball_joint: child leg_l_toe_a_ball -> leg_l_toe_a_ball_link
- joint leg_l_toe_a_link_joint: parent left_knee_pitch -> left_knee_pitch_link
- joint leg_l_toe_a_loop_joint: child leg_l_toe_a_loop -> leg_l_toe_a_loop_link; parent leg_l_toe_a_ball -> leg_l_toe_a_ball_link
- joint leg_l_toe_b_ball_joint: child leg_l_toe_b_ball -> leg_l_toe_b_ball_link
- joint leg_l_toe_b_link_joint: parent left_knee_pitch -> left_knee_pitch_link
- joint leg_l_toe_b_loop_joint: child leg_l_toe_b_loop -> leg_l_toe_b_loop_link; parent leg_l_toe_b_ball -> leg_l_toe_b_ball_link
- joint leg_r_toe_a_ball_joint: child leg_r_toe_a_ball -> leg_r_toe_a_ball_link
- joint leg_r_toe_a_link_joint: parent right_knee_pitch -> right_knee_pitch_link
- joint leg_r_toe_a_loop_joint: child leg_r_toe_a_loop -> leg_r_toe_a_loop_link; parent leg_r_toe_a_ball -> leg_r_toe_a_ball_link
- joint leg_r_toe_b_ball_joint: child leg_r_toe_b_ball -> leg_r_toe_b_ball_link
- joint leg_r_toe_b_link_joint: parent right_knee_pitch -> right_knee_pitch_link
- joint leg_r_toe_b_loop_joint: child leg_r_toe_b_loop -> leg_r_toe_b_loop_link; parent leg_r_toe_b_ball -> leg_r_toe_b_ball_link
- joint right_ankle_pitch_joint: child right_ankle_pitch -> right_ankle_pitch_link; limit lower=-3.14 upper=3.14 effort=80 velocity=10 -> lower=-0.41 upper=0.35 effort=80.0 velocity=13.61; parent right_knee_pitch -> right_knee_pitch_link
- joint right_ankle_roll_joint: child right_ankle_roll -> right_ankle_roll_link; limit lower=-3.14 upper=3.14 effort=80 velocity=10 -> lower=-0.64 upper=0.64 effort=80.0 velocity=13.61; parent right_ankle_pitch -> right_ankle_pitch_link
- joint right_elbow_pitch_joint: child right_elbow_pitch -> right_elbow_pitch_link; parent right_shoulder_yaw -> right_shoulder_yaw_link
- joint right_elbow_yaw_joint: child right_elbow_yaw -> right_elbow_yaw_link; parent right_elbow_pitch -> right_elbow_pitch_link
- joint right_hip_pitch_joint: child right_hip_pitch -> right_hip_pitch_link; limit lower=-3.14 upper=3.14 effort=150 velocity=8 -> lower=-2 upper=1 effort=180.0 velocity=8.9
- joint right_hip_roll_joint: child right_hip_roll -> right_hip_roll_link; limit lower=-3.14 upper=3.14 effort=150 velocity=8 -> lower=-0.2 upper=1.5 effort=150.0 velocity=27.23; parent right_hip_pitch -> right_hip_pitch_link
- joint right_hip_yaw_joint: child right_hip_yaw -> right_hip_yaw_link; limit lower=-3.14 upper=3.14 effort=50 velocity=24 -> lower=-1.5 upper=1.5 effort=150.0 velocity=27.23; origin xyz=0 -0.0777549159474913 0.0405999999999983 rpy=-1.57079632680723 0 0.00861027512635925 -> xyz=0 -0.0838049159474928 0.0405999999999983 rpy=-1.57079632680723 0 0; parent right_hip_roll -> right_hip_roll_link
- joint right_knee_pitch_joint: child right_knee_pitch -> right_knee_pitch_link; limit lower=-3.14 upper=3.14 effort=150 velocity=8 -> lower=0 upper=2 effort=180.0 velocity=8.9; origin xyz=-0.0347752157308957 0 -0.147956063988164 rpy=1.57940660192126 0 1.57079632822694 -> xyz=-0.0337000000000097 0 -0.142200000000001 rpy=1.5707963267949 0 1.5707963267949; parent right_hip_yaw -> right_hip_yaw_link
- joint right_shoulder_pitch_joint: child right_shoulder_pitch -> right_shoulder_pitch_link; parent lumber_pitch -> lumbar_pitch_link
- joint right_shoulder_roll_joint: child right_shoulder_roll -> right_shoulder_roll_link; parent right_shoulder_pitch -> right_shoulder_pitch_link
- joint right_shoulder_yaw_joint: child right_shoulder_yaw -> right_shoulder_yaw_link; parent right_shoulder_roll -> right_shoulder_roll_link
- joint right_wrist_pitch_joint: child right_wrist_pitch -> right_wrist_pitch_link; origin xyz=0.006 9.9998E-05 -0.1394 rpy=1.5708 0 0 -> xyz=0.006 0.0001 -0.1394 rpy=1.5708 0.229204 -1.5708; parent right_elbow_yaw -> right_elbow_yaw_link
- joint waist_motor_a_ball_joint: child waist_motor_a_ball -> waist_motor_a_ball_link
- joint waist_motor_a_link_joint: parent lumber_pitch -> lumbar_pitch_link
- joint waist_motor_a_loop_joint: child waist_motor_a_loop -> waist_motor_a_loop_link; parent waist_motor_a_ball -> waist_motor_a_ball_link
- joint waist_motor_b_ball_joint: child waist_motor_b_ball -> waist_motor_b_ball_link
- joint waist_motor_b_link_joint: parent lumber_pitch -> lumbar_pitch_link
- joint waist_motor_b_loop_joint: child waist_motor_b_loop -> waist_motor_b_loop_link; parent waist_motor_b_ball -> waist_motor_b_ball_link
